File: Project/Plates/Hull OEM 275u 225u.kicad_pcb (KiCad board)
At the start: 2 copper layers, 251.2 x 95.2 mm, 53 parts

Commit message: plate revisions
Parts:
- removed the REF** at (169.1, 134.9) (x2)
- removed the REF** at (121.4, 134.9) (x2)
- added REF**: Value, cipulot_parts:ecs_plate_cut_2U, F.Cu at (121.4, 134.9)
- added REF**: Value, cipulot_parts:ecs_plate_cut_2U, F.Cu at (169.1, 134.9)
Other:
- outline, holes or cut-outs redrawn
