File: Project/Plates/Hull OEM 625u.kicad_pcb (KiCad board)
At the start: 2 copper layers, 251.2 x 95.2 mm, 76 parts

Commit message: plate revisions
Parts:
- removed H1, H10, H11, H12, H13, H14, H15, H16, H17, H18, H19, H2, H20, H21, H22, H23, H24, H25, H26, H3, H4, H5, H6, H7, H8, H9: MountingHole, cipulot_parts:HOLE_M2
- removed the REF** at (154.8, 134.9)
- added REF**: Value, cipulot_parts:ecs_plate_cut_6.25U_space_stab, F.Cu at (154.8, 134.9)
- added REF**: Value, cipulot_parts:ecs_6.25U_space_stab, F.Cu at (154.8, 134.9)
Other:
- outline, holes or cut-outs redrawn
