File: Project/Plates/Hull 275u 225u MX.kicad_pcb (KiCad board)
At the start: 2 copper layers, 251.2 x 95.2 mm, 49 parts

Commit message: revision V1
changed bottom row mounting and boot cut for plates
Parts:
- added REF**: Value, cipulot_parts:ecs_plate_cut_2U, F.Cu at (169.1, 134.9)
- added REF**: Value, cipulot_parts:ecs_plate_cut_2U, F.Cu at (121.4, 134.9)
Other:
- outline, holes or cut-outs redrawn
- board text removed: "The Nicholas Van"
