File: Project/the-nicholas-van V1.kicad_pcb (KiCad board)
At the start: 4 copper layers, 242.9 x 95.2 mm, 143 parts, among them J1 JST SH, J2 Pico EZmate, J3 USB_C sink board 1.3mm, J4 Conn_01x05, J5 ARGB, SW1 BOOT0, U1 STM32F401CBUx, U2 XC6206PxxxMR, U3 74AHCT1G125, U4 74HC4051, U5 OPA350, U6 74HC4051, Y1 8 MHz

Commit message: v1 work
Parts:
- moved C16 5.97 mm to (34.9, 60.3), turned to 180 degrees
- moved C15 3.11 mm to (34.9, 54.8), turned to 180 degrees
- moved C17 2.98 mm to (34.9, 65.9), turned to 180 degrees
- moved J5 1.59 mm to (38.4, 51.6)
- moved C18 0.45 mm to (34.7, 69.0)
- moved U3 0.45 mm to (32.2, 68.6)
- moved J3 0.30 mm to (57.1, 51.1)
- moved R12 0.30 mm to (55.8, 58.1)
- moved R13 0.30 mm to (59.1, 58.1)
Routing:
- net +5V: track 93.7 -> 84.6 mm
- net COL0: track 172.8 -> 165.9 mm
- net COL5: track 147.0 -> 142.0 mm
- net ROW1: track 400.4 -> 396.7 mm
- net GND: track 99.6 -> 96.7 mm, vias 458 -> 453
- net ARGB: track 8.53 -> 5.57 mm, vias 2 -> 0
- net ROW2: track 384.5 -> 381.8 mm
- net COL6: track 102.9 -> 100.6 mm
- net Net-(LED2-DOUT): track 9.18 -> 7.74 mm
- net Net-(LED1-DOUT): track 9.18 -> 7.76 mm
- net APLEX_EN_PIN_1: track 72.7 -> 71.3 mm
- net COL11: track 167.7 -> 166.3 mm
- net D-: track 163.9 -> 162.6 mm
- net VBAT: track 313.9 -> 313.0 mm
- net ROW4: track 370.2 -> 369.4 mm
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Other:
- board text added: "JLCJLCJLCJLC"
