File: Project/analog.kicad_sch (KiCad schematic)
At the start: 22 parts, among them U4 74HC4051, U5 OPA350, U6 74HC4051

Commit message: backup
Other:
- moved on the sheet: C11, C12, C13, C14, JP1, R10, R15, R16, R17, R18, R19, R20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

Commit message: update revision
Parts:
- added C1: 100nF, Capacitor_SMD:C_0402_1005Metric, symbol Device:C
- added C2: 220pF NP0, Capacitor_SMD:C_0402_1005Metric, symbol Device:C
- added R1: 100k, Resistor_SMD:R_0402_1005Metric, symbol Device:R
- added R2: 1k, Resistor_SMD:R_0402_1005Metric, symbol Device:R
- added R3: DNP, Resistor_SMD:R_0402_1005Metric, symbol Device:R
- added U1: OPA354, Package_TO_SOT_SMD:SOT-23-5, symbol Amplifier_Operational:OPA340NA
Connections:
- net +3V3: now also C1.2, U1.5 (V+)
- net ADC: now also R1.1, R3.1, U1.1
- net GND: now also C1.1, C2.2, R2.2, U1.2 (V-)
- new net: R1.2, R2.1, R3.2, U1.4 (-)
- new net APLEX_OUT: C2.1, U1.3 (+)
Other:
- note added: "Alternatives: SC-70-6 OPA358AIDCKR LMV861 SOT-23-5 seems to have better availability OPA354 to 358 seems ok"
- note added: "placeholder for adjustment"
