File: Project/mounting.kicad_sch (KiCad schematic)
At the start: 28 parts

Commit message: fresh production files
Parts:
- removed H27, H28: MountingHole, cipulot_parts:HOLE_M2, symbol Mechanical:MountingHole
Changed lines of the file:
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@@
-    )
-  )
-  (symbol (lib_id "Mechanical:MountingHole") (at 35.56 127 0) (unit 1)
-    (in_bom yes) (on_board yes) (dnp no) (fields_autoplaced)
-    (property "Reference" "H27" (at 38.1 126.1653 0)
-      (effects (font (size 1.27 1.27)) (justify left))
-    )
-    (property "Value" "MountingHole" (at 38.1 128.7022 0)
-      (effects (font (size 1.27 1.27)) (justify left))
-    )
-    (property "Footprint" "cipulot_parts:HOLE_M2" (at 35.56 127 0)
-      (effects (font (size 1.27 1.27)) hide)
-    )
-    (property "Datasheet" "~" (at 35.56 127 0)
-      (effects (font (size 1.27 1.27)) hide)
-    )
-    (instances
-      (project "the-nicholas-van"
-        (path "/38f182bd-9097-4ce3-95d4-cd91b210c79b"
-          (reference "H27") (unit 1)
-        )
-        (path "/38f182bd-9097-4ce3-95d4-cd91b210c79b/610cabd0-87c8-472b-8f6a-63e84b5c9031"
-          (reference "H27") (unit 1)
-        )
-      )
-      (project "travaulta"
-        (path "/690df46b-b605-4617-b545-6aaced86d0fc/794114ef-7db2-4f90-86d0-13c32bb11aa3"
-          (reference "H17") (unit 1)
-        )
-      )
-      (project "EC60"
-        (path "/e63e39d7-6ac0-4ffd-8aa3-1841a4541b55/004107b0-ccf4-476d-9504-97bf1a9256af"
-          (reference "H1") (unit 1)
-        )
-      )
     )
   )
@@
         )
       )
-      (project "travaulta"
-        (path "/690df46b-b605-4617-b545-6aaced86d0fc/794114ef-7db2-4f90-86d0-13c32bb11aa3"
-          (reference "H17") (unit 1)
-        )
-      )
-      (project "EC60"
-        (path "/e63e39d7-6ac0-4ffd-8aa3-1841a4541b55/004107b0-ccf4-476d-9504-97bf1a9256af"
-          (reference "H1") (unit 1)
-        )
-      )
-    )
-  )
-  (symbol (lib_id "Mechanical:MountingHole") (at 60.96 127 0) (unit 1)
-    (in_bom yes) (on_board yes) (dnp no) (fields_autoplaced)
-    (property "Reference" "H28" (at 63.5 126.1653 0)
-      (effects (font (size 1.27 1.27)) (justify left))
-    )
-    (property "Value" "MountingHole" (at 63.5 128.7022 0)
-      (effects (font (size 1.27 1.27)) (justify left))
-    )
-    (property "Footprint" "cipulot_parts:HOLE_M2" (at 60.96 127 0)
-      (effects (font (size 1.27 1.27)) hide)
-    )
-    (property "Datasheet" "~" (at 60.96 127 0)
-      (effects (font (size 1.27 1.27)) hide)
-    )
-    (instances
-      (project "the-nicholas-van"
-        (path "/38f182bd-9097-4ce3-95d4-cd91b210c79b"
-          (reference "H28") (unit 1)
-        )
-        (path "/38f182bd-9097-4ce3-95d4-cd91b210c79b/610cabd0-87c8-472b-8f6a-63e84b5c9031"
-          (reference "H28") (unit 1)
-        )
-      )
